File: mx-pcb/Pteron36v0.kicad_pcb (KiCad board)
At the start: 2 copper layers, 131.3 x 104.9 mm, 63 parts, among them J1 AudioJack4, J2 AudioJack4, J3 Conn_01x04, SW10 SW_PUSH, SW12 SW_PUSH, SW13 SW_PUSH, SW14 SW_PUSH, SW15 SW_PUSH, SW17 SW_PUSH, SW18 SW_PUSH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

Commit message: First pass at 42 keys
Sent off to be made
Parts:
- added D1: 1N4148, Keebio-Parts:Diode-dual, F.Cu at (238.1, 78.9)
- added D2: 1N4148, Keebio-Parts:Diode-dual, F.Cu at (238.1, 96.0)
- added D3: 1N4148, Keebio-Parts:Diode-dual, F.Cu at (238.1, 115.7)
- added SW1: SW_PUSH, Keebio-Parts:Hybrid_PCB_100H_Dual_hole, F.Cu at (247.7, 76.9)
- added SW2: SW_PUSH, Keebio-Parts:Hybrid_PCB_100H_Dual_hole, F.Cu at (247.7, 95.9)
- added SW3: SW_PUSH, Keebio-Parts:Hybrid_PCB_100H_Dual_hole, F.Cu at (247.7, 115.0)
- moved D12 1.65 mm to (200.2, 67.3)
Connections:
- U1 pad 2: (no net) -> unconnected-(U1-RX-Pad2)
- U1 pad 24: (no net) -> unconnected-(U1-RAW-Pad24)
- U1 pad 7: (no net) -> unconnected-(U1-D4-Pad7)
- U1 pad 8: (no net) -> /Col6
Routing:
- net /Col6: track 0.00 -> 173.4 mm
- net /Row1: track 174.0 -> 191.5 mm
- net /Row3: track 266.6 -> 281.7 mm
- net Net-(D1-A): track 0.00 -> 12.2 mm
- net Net-(D3-A): track 0.00 -> 11.7 mm
- net Net-(D2-A): track 0.00 -> 11.0 mm
- net /Row2: track 327.3 -> 318.2 mm, vias 4 -> 6
- net /Col2: track 224.6 -> 229.6 mm
- net Net-(D18-A): track 30.3 -> 27.3 mm
- net SCL: track 29.7 -> 27.4 mm
- net SDA: track 36.6 -> 34.5 mm
- net /Col1: track 220.1 -> 221.9 mm
- net /Col4: track 124.2 -> 122.8 mm
- net Net-(D22-A): track 19.0 -> 18.2 mm
- net Net-(D12-A): track 22.0 -> 22.7 mm
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Other:
- board size 131.3 x 104.9 mm -> 149 x 103.9 mm
