File: mx-pcb/Pteron36v0.kicad_sch (KiCad schematic)
At the start: 63 parts, among them J1 AudioJack4, J2 AudioJack4, J3 Conn_01x04, SW10 SW_PUSH, SW12 SW_PUSH, SW13 SW_PUSH, SW14 SW_PUSH, SW15 SW_PUSH, SW17 SW_PUSH, SW18 SW_PUSH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

Commit message: First pass at 42 keys
Sent off to be made
Parts:
- added D1, D2, D3: 1N4148, Keebio-Parts:Diode-dual, symbol Diode:1N4148
- added SW1, SW2, SW3: SW_PUSH, Keebio-Parts:Hybrid_PCB_100H_Dual_hole, symbol keyboard_parts:SW_PUSH
Connections:
- net Row1: now also SW1.1
- net Row2: now also SW2.1
- net Row3: now also SW3.1
- net Col6: now reaches U1.8 (C6)
- net Col6: now also D1.1 (K), D2.1 (K), D3.1 (K)
- new net: D3.2 (A), SW3.2
- new net: D2.2 (A), SW2.2
- new net: D1.2 (A), SW1.2
- no-connect marks 4 -> 3
Other:
- moved on the sheet: D25, D_RE1, RE1, SW25
